Commit message: Add all updates.

File: src/vehicle_simulator/urdf/robot.urdf.xacro (robot description, xacro)
@@ -1,3 +1,4 @@
 <robot xmlns:xacro="http://www.ros.org/wiki/xacro" name="example">
+  <!-- 设置gazebo颜色的宏 -->
   <xacro:macro name="gazebo_material" params="ref color">
     <gazebo reference="${ref}">

File: src/velodyne_simulator/velodyne_description/urdf/VLP-16.urdf.xacro (robot description, xacro)
@@ -35,4 +35,5 @@
     <joint name="${name}_base_scan_joint" type="fixed" >
       <origin xyz="0 0 0.0377" rpy="0 0 0" />
+      <!-- <origin xyz="0.1 0 0.0377" rpy="0 0 0" /> -->
       <parent link="${name}_base_link" />
       <child link="${name}"/>
