Commit message: Add new models and worlds to p2os_urdf

File: src/p2os_urdf/defs/pioneer3at.xacro (robot description, xacro)
@@ -5,4 +5,5 @@
        xmlns:xacro="http://ros.org/wiki/xacro"
 name="pioneer3at">
+    <xacro:arg name="robot_namespace" default="robot_0"/>
     <xacro:property name="robot_namespace" value="$(arg robot_namespace)" />
     <!-- 惯性矩阵计算 -->

File: src/p2os_urdf/defs/pioneer3at_body.xacro (robot description, xacro)
@@ -5,5 +5,5 @@
        xmlns:xacro="http://ros.org/wiki/xacro"
 >
-    <xacro:arg name="robot_namespace" default=""/>
+    <!-- <xacro:arg name="robot_namespace" default=""/> -->
 <!-- Chassis -->
 	<link name="base_link">

File: src/p2os_urdf/defs/pioneer3at_without_3D.xacro (robot description, xacro)
@@ -22,5 +22,5 @@
         <child link="velodyne"/>
         <!-- 设置子link相对于父link的位姿 -->
-        <origin xyz="0 0 1" rpy="0 0 0"/>
+        <origin xyz="0 0 0.188" rpy="0 0 0"/>
     </joint>
     <xacro:p3at_front suffix="left" reflect="1"/>

File: src/p2os_urdf/defs/sensor_2D_laser.urdf.xacro (robot description, xacro)
@@ -1,5 +1,5 @@
 <robot name="2d_laser" xmlns:xacro="http://wiki.ros.org/xacro">
     <!--Gazebo Hokuyo Laser Plugin-->
-    <xacro:arg name="robot_namespace" default=""/>
+    <!-- <xacro:arg name="robot_namespace" default=""/> -->
     <gazebo reference="sensor_laser">
         <!-- <sensor type="gpu_ray" name="head_hokuyo_sensor"> -->
